File: 3 Way Adjustable Pot/3 Way Adjustable Pot.kicad_sch (KiCad schematic)
At the start: 31 parts, among them SW1 SW_MEC_5E, SW2 SW_MEC_5E, SW3 SW_MEC_5E, SW4 SW_MEC_5E, U1 74HC14, U2 74LS28, U3 74HC74, U4 74HC14, U5 CD74HC4066E, U6 74LS157, U7 LM555xN, U8 74LS139

Commit message: New KiCad intteration 2
Parts:
- added unit 5 of U4
Connections:
- net in_norm_off_rst: now also U4.3; no longer U3.1 (~{R}), U3.13 (~{R})
- net logic_!d0: now also U4.5; no longer U4.3
- net logic_!d1: now also U4.9; no longer U4.5
- net logic_!d3: now also U4.11; no longer U4.9
- net logic_d0: now also U4.6; no longer U4.4
- net logic_d1: now also U4.8; no longer U4.6
- net logic_d2: now also U4.10; no longer U4.8
- new net in_norm_on_rst: U3.1 (~{R}), U3.13 (~{R}), U4.4
Other:
- moved on the sheet: U4B, U4C, U4D
Changed lines of the file:
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@@
 		(title "Adjustable Digital Resistor")
 		(date "2025-12-10")
-		(rev "1")
+		(comment 1 "iteration 1")
 	)
 	(text "Push Buttons Inputs\n "
@@
 	(text "CMOS Tri-Switch\n"
 		(exclude_from_sim no)
-		(at 80.01 98.044 0)
+		(at 80.01 98.806 0)
 		(effects
 			(font
@@
 	(wire
 		(pts
+			(xy 116.84 74.93) (xy 116.84 68.58)
+		)
+		(stroke
+			(width 0)
+			(type default)
+		)
+	)
+	(wire
+		(pts
 			(xy 148.59 72.39) (xy 149.86 72.39)
 		)
@@
 	(wire
 		(pts
+			(xy 116.84 68.58) (xy 111.76 68.58)
+		)
+		(stroke
+			(width 0)
+			(type default)
+		)
+	)
+	(wire
+		(pts
 			(xy 135.89 34.29) (xy 127 34.29)
 		)
@@
 	(wire
 		(pts
+			(xy 90.17 66.04) (xy 76.2 66.04)
+		)
+		(stroke
+			(width 0)
+			(type default)
+		)
+	)
+	(wire
+		(pts
 			(xy 161.29 39.37) (xy 166.37 39.37)
 		)
@@
 	(wire
 		(pts
-			(xy 128.27 66.04) (xy 128.27 74.93)
-		)
-		(stroke
-			(width 0)
-			(type default)
-		)
-	)
-	(wire
-		(pts
 			(xy 66.04 124.46) (xy 57.15 124.46)
 		)
@@
 	(wire
 		(pts
-			(xy 87.63 62.23) (xy 90.17 62.23)
+			(xy 116.84 74.93) (xy 157.48 74.93)
 		)
 		(stroke
@@
 	(wire
 		(pts
-			(xy 128.27 43.18) (xy 118.11 43.18)
+			(xy 87.63 62.23) (xy 90.17 62.23)
 		)
 		(stroke
@@
 	(wire
 		(pts
-			(xy 157.48 74.93) (xy 128.27 74.93)
+			(xy 128.27 43.18) (xy 118.11 43.18)
 		)
 		(stroke
@@
 	(wire
 		(pts
-			(xy 76.2 66.04) (xy 128.27 66.04)
-		)
-		(stroke
-			(width 0)
-			(type default)
-		)
-	)
-	(wire
-		(pts
 			(xy 135.89 81.28) (xy 138.43 81.28)
 		)
@@
 	(wire
 		(pts
+			(xy 90.17 66.04) (xy 90.17 68.58)
+		)
+		(stroke
+			(width 0)
+			(type default)
+		)
+	)
+	(wire
+		(pts
 			(xy 182.88 74.93) (xy 182.88 76.2)
 		)
@@
 	(wire
 		(pts
+			(xy 96.52 68.58) (xy 90.17 68.58)
+		)
+		(stroke
+			(width 0)
+			(type default)
+		)
+	)
+	(wire
+		(pts
 			(xy 128.27 43.18) (xy 128.27 49.53)
 		)
@@
 		)
 	)
+	(label "in_norm_on_rst"
+		(at 118.11 74.93 0)
+		(effects
+			(font
+				(size 0.762 0.762)
+			)
+			(justify left bottom)
+		)
+	)
 	(label "in_norm_off_2"
 		(at 77.47 50.8 0)
@@
 	(symbol
 		(lib_id "74xx:74HC14")
-		(at 123.19 133.35 0)
+		(at 115.57 121.92 0)
 		(mirror y)
 		(unit 4)
@@
 		(fields_autoplaced yes)
 		(property "Reference" "U4"
-			(at 123.19 124.46 0)
+			(at 115.57 113.03 0)
 			(effects
 				(font
@@
 		)
 		(property "Value" "74HC14"
-			(at 123.19 127 0)
+			(at 115.57 115.57 0)
 			(effects
 				(font
@@
 		)
 		(property "Footprint" ""
-			(at 123.19 133.35 0)
+			(at 115.57 121.92 0)
 			(effects
 				(font
@@
 		)
 		(property "Datasheet" "http://www.ti.com/lit/gpn/sn74HC14"
-			(at 123.19 133.35 0)
+			(at 115.57 121.92 0)
 			(effects
 				(font
@@
 		)
 		(property "Description" "Hex inverter schmitt trigger"
-			(at 123.19 133.35 0)
+			(at 115.57 121.92 0)
 			(effects
 				(font
@@
 	(symbol
 		(lib_id "74xx:74HC14")
-		(at 107.95 110.49 180)
+		(at 104.14 68.58 0)
 		(unit 2)
 		(exclude_from_sim no)
@@
 		(on_board yes)
 		(dnp no)
-		(fields_autoplaced yes)
 		(property "Reference" "U4"
-			(at 107.95 101.6 0)
+			(at 103.886 72.644 0)
 			(effects
 				(font
@@
 		)
 		(property "Value" "74HC14"
-			(at 107.95 104.14 0)
+			(at 103.886 75.184 0)
 			(effects
 				(font
@@
 		)
 		(property "Footprint" ""
-			(at 107.95 110.49 0)
+			(at 104.14 68.58 0)
 			(effects
 				(font
@@
 		)
 		(property "Datasheet" "http://www.ti.com/lit/gpn/sn74HC14"
-			(at 107.95 110.49 0)
+			(at 104.14 68.58 0)
 			(effects
 				(font
@@
 		)
 		(property "Description" "Hex inverter schmitt trigger"
-			(at 107.95 110.49 0)
+			(at 104.14 68.58 0)
 			(effects
 				(font
@@
 	(symbol
 		(lib_id "74xx:74HC14")
-		(at 115.57 121.92 180)
+		(at 107.95 110.49 180)
 		(unit 3)
 		(exclude_from_sim no)
@@
 		(fields_autoplaced yes)
 		(property "Reference" "U4"
-			(at 115.57 113.03 0)
+			(at 107.95 101.6 0)
 			(effects
 				(font
@@
 		)
 		(property "Value" "74HC14"
-			(at 115.57 115.57 0)
+			(at 107.95 104.14 0)
 			(effects
 				(font
@@
 		)
 		(property "Footprint" ""
-			(at 115.57 121.92 0)
+			(at 107.95 110.49 0)
 			(effects
 				(font
@@
 		)
 		(property "Datasheet" "http://www.ti.com/lit/gpn/sn74HC14"
-			(at 115.57 121.92 0)
+			(at 107.95 110.49 0)
 			(effects
 				(font
@@
 		)
 		(property "Description" "Hex inverter schmitt trigger"
-			(at 115.57 121.92 0)
+			(at 107.95 110.49 0)
 			(effects
 				(font
@@
 				)
 			)
+		)
+	)
+	(symbol
+		(lib_id "74xx:74HC14")
+		(at 123.19 133.35 180)
+		(unit 5)
+		(exclude_from_sim no)
+		(in_bom yes)
+		(on_board yes)
+		(dnp no)
+		(fields_autoplaced yes)
+		(property "Reference" "U4"
+			(at 123.19 124.46 0)
+			(effects
+				(font
+					(size 1.27 1.27)
+				)
+			)
+		)
+		(property "Value" "74HC14"
+			(at 123.19 127 0)
+			(effects
+				(font
+					(size 1.27 1.27)
+				)
+			)
+		)
+		(property "Footprint" ""
+			(at 123.19 133.35 0)
+			(effects
+				(font
+					(size 1.27 1.27)
+				)
+				(hide yes)
+			)
+		)
+		(property "Datasheet" "http://www.ti.com/lit/gpn/sn74HC14"
+			(at 123.19 133.35 0)
+			(effects
+				(font
+					(size 1.27 1.27)
+				)
+				(hide yes)
+			)
+		)
+		(property "Description" "Hex inverter schmitt trigger"
+			(at 123.19 133.35 0)
+			(effects
+				(font
+					(size 1.27 1.27)
+				)
+				(hide yes)
+			)
+		)
+		(pin "1"
+		)
+		(pin "2"
+		)
+		(pin "13"
+		)
+		(pin "14"
+		)
+		(pin "4"
+		)
+		(pin "7"
+		)
+		(pin "12"
+		)
+		(pin "3"
+		)
+		(pin "9"
+		)
+		(pin "8"
+		)
+		(pin "10"
+		)
+		(pin "5"
+		)
+		(pin "6"
+		)
+		(pin "11"
+		)
+		(instances
+			(project ""
+				(path "/51f00b6a-0452-4345-b95d-48d0ef48a867"
+					(reference "U4")
+					(unit 5)
+				)
+			)
